Commit message: revert urdf to match the exact xarm7 kinematics

File: xarm_description/urdf/xarm7/xarm7.urdf.xacro (robot description, xacro)
@@ -74,34 +74,4 @@
       </collision>
     </link>
-    <link name="${prefix}wall_plane_1">
-      <visual>
-        <origin xyz="0.0 0.0 0.0" rpy="0.0 0.0 0.0"/>
-        <geometry>
-          <mesh filename="package://xarm_description/meshes/xarm7/visual/table_plane.stl" scale="0.0001 0.0001 0.0005"/>
-        </geometry>
-        <material name="Wall"/>
-      </visual>
-      <collision>
-        <origin xyz="0.0 0.0 0.0" rpy="0.0 0.0 0.0"/>
-        <geometry>
-          <mesh filename="package://xarm_description/meshes/xarm7/visual/table_plane.stl" scale="0.0001 0.0001 0.0005"/>
-        </geometry>
-      </collision>
-    </link>
-    <link name="${prefix}wall_plane_2">
-      <visual>
-        <origin xyz="0.0 0.0 0.0" rpy="0.0 0.0 0.0"/>
-        <geometry>
-          <mesh filename="package://xarm_description/meshes/xarm7/visual/table_plane.stl" scale="0.0001 0.0001 0.0005"/>
-        </geometry>
-        <material name="Wall"/>
-      </visual>
-      <collision>
-        <origin xyz="0.0 0.0 0.0" rpy="0.0 0.0 0.0"/>
-        <geometry>
-          <mesh filename="package://xarm_description/meshes/xarm7/visual/table_plane.stl" scale="0.0001 0.0001 0.0005"/>
-        </geometry>
-      </collision>
-    </link>
     <joint name="${prefix}link_base_table_plane_joint" type="fixed">
       <origin xyz="0.7 -0.6 -0.01" rpy="0.0 0.0 1.5708"/>
@@ -109,15 +79,4 @@
       <parent link="world"/>
       <child link="${prefix}table_plane"/>
-    </joint>
-    <joint name="${prefix}link_base_wall_plane_1_joint" type="fixed">
-      <!-- <origin xyz="-0.3 -0.6 0.00" rpy="1.5708 0.0 1.5708"/> -->
-      <origin xyz="-0.15 -0.6 0.05" rpy="1.5708 0.0 1.5708"/>
-      <parent link="world"/>
-      <child link="${prefix}wall_plane_1"/>
-    </joint>
-    <joint name="${prefix}link_base_wall_plane_2_joint" type="fixed">
-      <origin xyz="-0.1 -0.6 0.705" rpy="3.142 0.0 1.5708"/>
-      <parent link="world"/>
-      <child link="${prefix}wall_plane_2"/>
     </joint>
     <link name="${prefix}link_base">
@@ -221,11 +180,9 @@
       <child link="${prefix}link3" />
       <axis xyz="0 0 1" />
-      <!-- <limit
+      <limit
         lower="${joint3_lower_limit}"
         upper="${joint3_upper_limit}"
         effort="30"
-        velocity="3.14" /> -->
-        <limit lower="${-0.035}" upper="${0.035}" effort="30" velocity="3.14" />
-      <dynamics damping="5" friction="1" />
+        velocity="3.14" />
     </joint>
     <link name="${prefix}link4">

Commit message: edit: removed the wall links,

File: xarm_description/urdf/xarm7/xarm7.urdf.xacro (robot description, xacro)
@@ -55,8 +55,5 @@
       <color rgba="0.55 0.27 0.07 1.0"/>
     </material>
-    <material name="Wall">
-      <color rgba="0.98 0.97 0.95 1.0"/>
-    </material>
-        <!-- Table plane to assist in collision detection and thus in trajectory generation  -->
+        <!-- Table plane to assist in collision detection and thus in trajectory planning and generation  -->
     <link name="${prefix}table_plane">
       <visual>
